File: MagnetorquerSidePanels/Coil_Panels_XY.kicad_pcb (KiCad board)
At the start: 6 copper layers, 82 x 108 mm, 15 parts, among them J1 Through_Hole_1, J2 MOLEX_2053380006

Commit message: added 3D models to magnetorquer side panel boards
Parts:
- J2: value MOLEX_2053380006 -> Conn_01x06
Changed lines of the file:
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@@
         (effects (font (size 1 1) (thickness 0.15)) (justify mirror))
     )
-    (fp_text value "MOLEX_2053380006" (at 1.66 -6.415 90) (layer "B.Fab")
+    (fp_text value "Conn_01x06" (at 1.66 -6.415 90) (layer "B.Fab")
         (effects (font (size 1 1) (thickness 0.15)) (justify mirror))
     )
@@
     (pad "S2" smd rect (at -7.895 2.425 90) (size 1.35 2.9) (layers "B.Cu" "B.Paste")
       (net 13 "unconnected-(J2-SHIELD2-PadS2)") (pinfunction "SHIELD2") (pintype "no_connect"))
-    (model "${KIPRJMOD}/cad/2053380006.stp"
+    (model "${SAMWISE_AVIONICS}/3D_models/panels/2053380006.step"
       (offset (xyz 0 1.5 1.3))
       (scale (xyz 1 1 1))
