File: MagnetorquerSidePanels/_autosave-Z_Panels.kicad_pcb (KiCad board)
At the start: 4 copper layers, 97 x 97.3 mm, 36 parts, among them J1 SMA Connector Male, J2 Conn_01x04_MountingPin, J4 Conn_01x04_MountingPin, U1 LTC2051IS8_PBF, U2 HHM1589D1

Commit message: pre-board review
Routing:
- net OUT1: track 78.9 -> 94.1 mm, vias 2 -> 5
- net OUT2: track 70.9 -> 80.4 mm
- net +3V3: track 62.1 -> 63.6 mm
- net /Photodiode 1/IN-: track 32.6 -> 33.2 mm
Changed lines of the file:
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@@
   (segment (start 202.552 88.44) (end 195.84 88.44) (width 0.25) (layer "F.Cu") (net 11))
   (segment (start 195.84 88.44) (end 195.8 88.4) (width 0.25) (layer "F.Cu") (net 11))
+  (segment (start 179.9 107.975) (end 180.925 107.975) (width 0.25) (layer "F.Cu") (net 13))
   (segment (start 165.575 109.175) (end 178.7 109.175) (width 0.25) (layer "F.Cu") (net 13))
   (segment (start 164.35 105.45) (end 164.35 107.95) (width 0.25) (layer "F.Cu") (net 13))
-  (segment (start 181.485 106.39) (end 181.485 105.0233) (width 0.25) (layer "F.Cu") (net 13))
+  (segment (start 180.925 107.975) (end 181.485 107.415) (width 0.25) (layer "F.Cu") (net 13))
+  (segment (start 178.7 109.175) (end 179.9 107.975) (width 0.25) (layer "F.Cu") (net 13))
   (segment (start 164.35 107.95) (end 165.575 109.175) (width 0.25) (layer "F.Cu") (net 13))
-  (segment (start 178.7 109.175) (end 181.485 106.39) (width 0.25) (layer "F.Cu") (net 13))
+  (segment (start 181.485 107.415) (end 181.485 105.0233) (width 0.25) (layer "F.Cu") (net 13))
   (via (at 178.7 109.175) (size 0.8) (drill 0.4) (layers "F.Cu" "B.Cu") (net 13))
   (segment (start 179.125 109.6) (end 178.7 109.175) (width 0.25) (layer "B.Cu") (net 13))
@@
   (segment (start 188.475 109.55) (end 184.625 109.55) (width 0.25) (layer "B.Cu") (net 13))
   (segment (start 190.25 108.1) (end 190.25 65.25) (width 0.25) (layer "F.Cu") (net 15))
+  (segment (start 183.175 111.925) (end 183.175 107.9) (width 0.25) (layer "F.Cu") (net 15))
+  (segment (start 181.775 113.325) (end 183.175 111.925) (width 0.25) (layer "F.Cu") (net 15))
+  (segment (start 179.225 106.0133) (end 180.215 105.0233) (width 0.25) (layer "F.Cu") (net 15))
   (segment (start 177.6 52.6) (end 174.625 52.6) (width 0.25) (layer "F.Cu") (net 15))
   (segment (start 190.25 65.25) (end 177.6 52.6) (width 0.25) (layer "F.Cu") (net 15))
+  (segment (start 179.225 106.8) (end 179.225 106.0133) (width 0.25) (layer "F.Cu") (net 15))
   (segment (start 174.625 52.6) (end 173.075 54.15) (width 0.25) (layer "F.Cu") (net 15))
+  (via (at 183.175 107.9) (size 0.8) (drill 0.4) (layers "F.Cu" "B.Cu") (net 15))
+  (via (at 181.775 113.325) (size 0.8) (drill 0.4) (layers "F.Cu" "B.Cu") (net 15))
+  (via (at 179.225 106.8) (size 0.8) (drill 0.4) (layers "F.Cu" "B.Cu") (net 15))
   (via (at 173.075 54.15) (size 0.8) (drill 0.4) (layers "F.Cu" "B.Cu") (net 15))
   (via (at 190.25 108.1) (size 0.8) (drill 0.4) (layers "F.Cu" "B.Cu") (net 15))
   (segment (start 184.6 111.125) (end 188.4 111.125) (width 0.25) (layer "B.Cu") (net 15))
   (segment (start 188.475 111.2) (end 190.25 109.425) (width 0.25) (layer "B.Cu") (net 15))
+  (segment (start 183.175 107.9) (end 180.325 107.9) (width 0.25) (layer "B.Cu") (net 15))
+  (segment (start 180.325 107.9) (end 179.225 106.8) (width 0.25) (layer "B.Cu") (net 15))
+  (segment (start 180.85 112.4) (end 181.775 113.325) (width 0.25) (layer "B.Cu") (net 15))
+  (segment (start 180.85 111.15) (end 180.85 112.4) (width 0.25) (layer "B.Cu") (net 15))
   (segment (start 173.075 55.6) (end 173.125 55.65) (width 0.25) (layer "B.Cu") (net 15))
   (segment (start 184.575 111.15) (end 184.6 111.125) (width 0.25) (layer "B.Cu") (net 15))
@@
   (via (at 177.15 56.075) (size 0.8) (drill 0.4) (layers "F.Cu" "B.Cu") (net 17))
   (via (at 186.375 64.525) (size 0.8) (drill 0.4) (layers "F.Cu" "B.Cu") (net 17))
-  (segment (start 190.075 99.75) (end 190.075 68.225) (width 0.25) (layer "B.Cu") (net 17))
+  (segment (start 188.05 93) (end 190.075 93) (width 0.25) (layer "B.Cu") (net 17))
   (segment (start 175.550001 56.075) (end 175.125001 55.65) (width 0.25) (layer "B.Cu") (net 17))
   (segment (start 190.075 68.225) (end 186.375 64.525) (width 0.25) (layer "B.Cu") (net 17))
   (segment (start 188.015 101.81) (end 190.075 99.75) (width 0.25) (layer "B.Cu") (net 17))
+  (segment (start 190.075 93) (end 190.075 68.225) (width 0.25) (layer "B.Cu") (net 17))
   (segment (start 177.15 56.075) (end 175.550001 56.075) (width 0.25) (layer "B.Cu") (net 17))
   (segment (start 184.35 93) (end 180.55 93) (width 0.25) (layer "B.Cu") (net 17))
+  (segment (start 180.55 93) (end 188.05 93) (width 0.25) (layer "B.Cu") (net 17))
   (segment (start 188.05 93) (end 184.35 93) (width 0.25) (layer "B.Cu") (net 17))
   (segment (start 181.485 101.81) (end 188.015 101.81) (width 0.25) (layer "B.Cu") (net 17))
-  (segment (start 179.975 60.625) (end 172.5 60.625) (width 0.25) (layer "F.Cu") (net 18))
-  (segment (start 180.2375 97.5875) (end 188.575 89.25) (width 0.25) (layer "F.Cu") (net 18))
+  (segment (start 190.075 99.75) (end 190.075 93) (width 0.25) (layer "B.Cu") (net 17))
+  (segment (start 181.8 96.025) (end 185.8 96.025) (width 0.25) (layer "F.Cu") (net 18))
+  (segment (start 180.2375 97.5875) (end 181.8 96.025) (width 0.25) (layer "F.Cu") (net 18))
+  (segment (start 175 55.65) (end 167.525 55.65) (width 0.25) (layer "F.Cu") (net 18))
+  (segment (start 187.575 68.225) (end 175 55.65) (width 0.25) (layer "F.Cu") (net 18))
   (segment (start 180.2375 97.5875) (end 180.215 97.61) (width 0.25) (layer "F.Cu") (net 18))
+  (segment (start 187.575 94.25) (end 187.575 68.225) (width 0.25) (layer "F.Cu") (net 18))
   (segment (start 180.215 97.61) (end 180.215 99.575) (width 0.25) (layer "F.Cu") (net 18))
-  (segment (start 172.5 60.625) (end 167.525 55.65) (width 0.25) (layer "F.Cu") (net 18))
-  (segment (start 188.575 89.25) (end 188.575 69.225) (width 0.25) (layer "F.Cu") (net 18))
-  (segment (start 188.575 69.225) (end 179.975 60.625) (width 0.25) (layer "F.Cu") (net 18))
+  (segment (start 185.8 96.025) (end 187.575 94.25) (width 0.25) (layer "F.Cu") (net 18))
   (via (at 180.2375 97.5875) (size 0.8) (drill 0.4) (layers "F.Cu" "B.Cu") (net 18))
   (via (at 167.525 55.65) (size 0.8) (drill 0.4) (layers "F.Cu" "B.Cu") (net 18))
