File: New_Coil_Panel_Y/New_Coil_Panel_Y.kicad_pcb (KiCad board)
At the start: 6 copper layers, 215.5 x 81.5 mm, 9 parts, among them J1 CON_2053380002

Commit message: added gerbers, name
Other:
- board text added: "Eric Liu"
Changed lines of the file:
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@@
       (plot_on_all_layers_selection 0x0000000_00000000)
       (disableapertmacros false)
-      (usegerberextensions false)
+      (usegerberextensions true)
       (usegerberattributes true)
-      (usegerberadvancedattributes true)
+      (usegerberadvancedattributes false)
       (creategerberjobfile true)
       (dashed_line_dash_ratio 12.000000)
@@
       (psa4output false)
       (plotreference true)
-      (plotvalue true)
+      (plotvalue false)
       (plotinvisibletext false)
       (sketchpadsonfab false)
-      (subtractmaskfromsilk false)
+      (subtractmaskfromsilk true)
       (outputformat 1)
       (mirror false)
-      (drillshape 1)
+      (drillshape 0)
       (scaleselection 1)
-      (outputdirectory "")
+      (outputdirectory "gerbers_Y_fixed_20240308/")
     )
   )
@@
         (effects (font (size 1 1) (thickness 0.15)))
     )
-    (fp_text user "*" (at 0 0 90) (layer "B.SilkS")
-        (effects (font (size 1 1) (thickness 0.15)) (justify mirror))
-    )
     (fp_text user "Copyright 2021 Accelerated Designs. All rights reserved." (at 0 0 90) (layer "Cmts.User")
         (effects (font (size 0.127 0.127) (thickness 0.002)))
@@
   (gr_line locked (start 264.65 52.578) (end 264.65 53.001216)
     (stroke (width 0.2) (type solid)) (layer "Edge.Cuts"))
+  (gr_text "Eric Liu" (at 271.396 120.554 90) (layer "F.SilkS")
+    (effects (font (size 1.5 1.5) (thickness 0.3) bold) (justify left bottom))
+  )
   (segment (start 109.708 90.17) (end 111.712178 90.17) (width 0.305) (layer "B.Cu") (net 7))
   (segment (start 113.535 82.297499) (end 111.5 80.262499) (width 0.305) (layer "B.Cu") (net 7))
