File: BatteryBoard/batteryboard-v02b/batteryboard.kicad_pcb (KiCad board)
At the start: 4 copper layers, 95.9 x 90.2 mm, 40 parts, among them J1 KEYSTONE-1042, J2 KEYSTONE-1042, J3 KEYSTONE-1042, J4 KEYSTONE-1042, J5 KEYSTONE-1042, J6 KEYSTONE-1042, J7 MOLEX 502352-0801, J8 Screw_Terminal_01x02, Q1 IRF7458, Q2 IRF7458, Q4 IRLML2803, U1 R5460N233AF, U2 DMP2040USS-13

Commit message: cleaned up ibom, footprints
Parts:
- J7: footprint batteryboard_local:CONN_502352-0801_MOL -> batteryboard:502352-0801
- R10: value 100k -> 100K
- R6: value 200k, RN73H2BTTD2003A05 -> 200K, RN73H2BTTD2003A05
- R8: value 10k -> 10K
- R9: value 4.7k -> 4.7K
Other:
- board text added: "Heater_ Enable"
- board text added: "Temp_ Sense"
- board text removed: "Enable"
- board text removed: "Sense"
Changed lines of the file:
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@@
     (property "Sheetfile" "batteryboard.kicad_sch")
     (property "Sheetname" "")
+    (property "exclude_from_bom" "")
     (property "ki_description" "test point")
     (property "ki_keywords" "test point tp")
-    (attr through_hole)
+    (attr through_hole exclude_from_bom)
     (fp_text reference "TP1" (at 0.7 2.5) (layer "F.SilkS") hide
         (effects (font (size 1 1) (thickness 0.15)))
@@
     (property "Sheetfile" "batteryboard.kicad_sch")
     (property "Sheetname" "")
+    (property "exclude_from_bom" "")
     (property "ki_description" "test point")
     (property "ki_keywords" "test point tp")
-    (attr through_hole)
+    (attr through_hole exclude_from_bom)
     (fp_text reference "TP2" (at 0.7 2.5) (layer "F.SilkS") hide
         (effects (font (size 1 1) (thickness 0.15)))
@@
         (effects (font (size 1 1) (thickness 0.15)))
     )
-    (fp_text value "200k, RN73H2BTTD2003A05" (at 0 1.82 90) (layer "F.Fab")
+    (fp_text value "200K, RN73H2BTTD2003A05" (at 0 1.82 90) (layer "F.Fab")
         (effects (font (size 1 1) (thickness 0.15)))
     )
@@
         (effects (font (size 1 1) (thickness 0.15)))
     )
-    (fp_text value "10k" (at 0 1.43) (layer "F.Fab")
+    (fp_text value "10K" (at 0 1.43) (layer "F.Fab")
         (effects (font (size 1 1) (thickness 0.15)))
     )
@@
         (effects (font (size 0.8 0.9) (thickness 0.15)))
     )
-    (fp_text value "4.7k" (at 0 1.43) (layer "F.Fab")
+    (fp_text value "4.7K" (at 0 1.43) (layer "F.Fab")
         (effects (font (size 1 1) (thickness 0.15)))
     )
@@
       (net 18 "/HEATER") (pinfunction "2") (pintype "passive"))
   )
-  (footprint "batteryboard_local:CONN_502352-0801_MOL" (layer "F.Cu")
+  (footprint "batteryboard:502352-0801" (layer "F.Cu")
     (at 88.6803 67.6799 180)
     (tags "502352-0801 ")
@@
     (property "ki_keywords" "502352-0801")
     (attr smd)
-    (fp_text reference "J7" (at 12.2606 -4.574 unlocked) (layer "F.SilkS")
+    (fp_text reference "J7" (at 12.3356 -4.549 unlocked) (layer "F.SilkS")
         (effects (font (size 1 1) (thickness 0.15)))
     )
@@
         (effects (font (size 0.8 0.9) (thickness 0.15)))
     )
-    (fp_text value "100k" (at 0 1.43) (layer "F.Fab")
+    (fp_text value "100K" (at 0 1.43) (layer "F.Fab")
         (effects (font (size 1 1) (thickness 0.15)))
     )
@@
     (effects (font (size 1.2 1.2) (thickness 0.2)))
   )
-  (gr_text "Enable" (at 91.6395 75.3041 90) (layer "F.SilkS")
+  (gr_text "Heater_\nEnable" (at 89.7447 75.4789 90) (layer "F.SilkS")
     (effects (font (size 0.8 0.8) (thickness 0.15)))
   )
-  (gr_text "Sense" (at 89.5567 74.9485 90) (layer "F.SilkS")
+  (gr_text "Temp_\nSense" (at 91.8447 75.1289 90) (layer "F.SilkS")
     (effects (font (size 0.8 0.8) (thickness 0.15)))
   )

Commit message: changed kilo to lowercase
Parts:
- R10: value 100K -> 100k
- R4: value 1K -> 1k
- R6: value 200K, RN73H2BTTD2003A05 -> 200k, RN73H2BTTD2003A05
- R8: value 10K -> 10k
- R9: value 4.7K -> 4.7k
Changed lines of the file:
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@@
         (effects (font (size 1 1) (thickness 0.15)))
     )
-    (fp_text value "1K" (at 0 1.43 90) (layer "F.Fab")
+    (fp_text value "1k" (at 0 1.43 90) (layer "F.Fab")
         (effects (font (size 1 1) (thickness 0.15)))
     )
@@
         (effects (font (size 1 1) (thickness 0.15)))
     )
-    (fp_text value "200K, RN73H2BTTD2003A05" (at 0 1.82 90) (layer "F.Fab")
+    (fp_text value "200k, RN73H2BTTD2003A05" (at 0 1.82 90) (layer "F.Fab")
         (effects (font (size 1 1) (thickness 0.15)))
     )
@@
         (effects (font (size 1 1) (thickness 0.15)))
     )
-    (fp_text value "10K" (at 0 1.43) (layer "F.Fab")
+    (fp_text value "10k" (at 0 1.43) (layer "F.Fab")
         (effects (font (size 1 1) (thickness 0.15)))
     )
@@
         (effects (font (size 0.8 0.9) (thickness 0.15)))
     )
-    (fp_text value "4.7K" (at 0 1.43) (layer "F.Fab")
+    (fp_text value "4.7k" (at 0 1.43) (layer "F.Fab")
         (effects (font (size 1 1) (thickness 0.15)))
     )
@@
         (effects (font (size 0.8 0.9) (thickness 0.15)))
     )
-    (fp_text value "100K" (at 0 1.43) (layer "F.Fab")
+    (fp_text value "100k" (at 0 1.43) (layer "F.Fab")
         (effects (font (size 1 1) (thickness 0.15)))
     )
