File: BatteryBoard/batteryboard-v02c/batteryboard.kicad_sch (KiCad schematic)
At the start: 36 parts, among them J1 KEYSTONE-1042, J2 KEYSTONE-1042, J3 KEYSTONE-1042, J4 KEYSTONE-1042, J5 KEYSTONE-1042, J6 KEYSTONE-1042, J7 MOLEX 502352-0801, J8 1985807, Q1 IRF7458, Q2 IRF7458, Q3 DMP2040USS-13, Q4 IRLML2803, U1 R5460N233AF

Commit message: changed flags
Connections:
- net PyCubed_AIN5 renamed PyCubed_SENSE
- net PyCubed_HIN renamed PyCubed_ENABLE
