File: ADCS/ADCS_board/watchdog.kicad_sch (KiCad schematic)
At the start: 28 parts, among them U7 TLV1704

Commit message: main adcs board with initial traces coming out of MCU
Other:
- title: PyCubed Mainboard -> Watchdog
Changed lines of the file:
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@@
 	(paper "USLetter")
 	(title_block
-		(title "PyCubed Mainboard")
+		(title "Watchdog")
 		(date "2024-11-24")
-		(rev "v06c")
+		(rev "v1")
 		(company "Stanford Student Space Initiative")
 		(comment 1 "Ethan Brinser")
+		(comment 2 "From PiCubed")
 	)
 	(junction
