File: ADCS/ADCS-v0-samwise/GPS.kicad_sch (KiCad schematic)
At the start: 5 parts, among them J7 Amphenol_901-144, J8 Amphenol_901-144, U12 Orion B16, U13 EP2W+

Commit message: incorporated first round of feedbacks
Parts:
- R35: footprint Resistor_SMD:R_0402_1005Metric -> Resistor_SMD:R_0603_1608Metric
Connections:
- net V_BCKP is gone; now on net 3V3_GPS: U12.22 (V_BCKP)
Changed lines of the file:
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@@
+	)
+	(junction
+		(at 128.27 120.65)
+		(diameter 0)
+		(color 0 0 0 0)
 	)
 	(junction
@@
 	(wire
 		(pts
+			(xy 152.4 118.11) (xy 128.27 118.11)
+		)
+		(stroke
+			(width 0)
+			(type default)
+		)
+	)
+	(wire
+		(pts
 			(xy 193.04 66.04) (xy 193.04 95.25)
 		)
@@
 	(wire
 		(pts
+			(xy 128.27 120.65) (xy 152.4 120.65)
+		)
+		(stroke
+			(width 0)
+			(type default)
+		)
+	)
+	(wire
+		(pts
 			(xy 200.66 102.87) (xy 200.66 107.95)
 		)
@@
 	(wire
 		(pts
-			(xy 115.57 120.65) (xy 152.4 120.65)
+			(xy 115.57 120.65) (xy 128.27 120.65)
 		)
 		(stroke
@@
 		(pts
 			(xy 226.06 76.2) (xy 241.3 76.2)
+		)
+		(stroke
+			(width 0)
+			(type default)
+		)
+	)
+	(wire
+		(pts
+			(xy 128.27 118.11) (xy 128.27 120.65)
 		)
 		(stroke
@@
 				(hide yes)
 			)
-		)
-	)
-	(hierarchical_label "V_BCKP"
-		(shape input)
-		(at 152.4 118.11 180)
-		(fields_autoplaced yes)
-		(effects
-			(font
-				(size 1.27 1.27)
-			)
-			(justify right)
 		)
 	)
@@
 			)
 		)
-		(property "Footprint" "Resistor_SMD:R_0402_1005Metric"
+		(property "Footprint" "Resistor_SMD:R_0603_1608Metric"
 			(at 209.55 107.95 0)
 			(effects
