File: ADCS/ADCS-v0-samwise/magnetorquer_driver.kicad_sch (KiCad schematic)
At the start: 33 parts, among them U1 MP6551GQB-P, U6 MP6551GQB-P, U8 MP6551GQB-P

Commit message: incorporated first round of feedbacks
Parts:
- removed C24, C33, C9: 470u, Capacitor_SMD:C_0603_1608Metric, symbol Device:C_Polarized_US
- added C24, C33, C9: 22u, Capacitor_SMD:C_0603_1608Metric, symbol Device:C
Connections:
- net GND: now also C24.2, C33.2, C9.2
- net VBATT_REG: now also C24.1, C33.1, C9.1
