File: ADCS/ADCS-v01b-samwise/Connectors.kicad_sch (KiCad schematic)
At the start: 19 parts, among them J11 Conn_01x10, J13 USB_C_pycubed, J14 2053380002, J15 2053380002, J16 2053380002, J2 Conn_ARM_JTAG_SWD_10, J22 QWIIC, J5 35362-1250, J6 Conn_01x04

Commit message: Changes to ADCS board as of 20250322
Parts:
- removed R59, R71: 10k, Resistor_SMD:R_0603_1608Metric, symbol Device:R_US
- added J13, J14, J15: 2053380002, ssi_connector:Molex_205338-0002, symbol ssi_connector:205338-0002
- JP1: renamed from JP5; value QWIIC suply -> QWIIC supply
- renumbered J14 to J10, J15 to J11, J16 to J12, J22 to J19, J2 to J20, J5 to J4, J6 to J5, J11 to J8, J13 to J9
Connections:
- net VBATT_SENSE: no longer J8.5 (Pin_5), J8.7 (Pin_7), J8.9 (Pin_9)
- net X_MAGDRV_OUT1: now also J10.1, J13.2; no longer J11.1
- net X_MAGDRV_OUT2: now also J10.2, J13.1; no longer J11.2
- net Y_MAGDRV_OUT1: now also J11.1, J14.2; no longer J12.1
- net Y_MAGDRV_OUT2: now also J11.2, J14.1; no longer J12.2
- net Z_MAGDRV_OUT1: now also J12.1, J15.2; no longer J10.1
- net Z_MAGDRV_OUT2: now also J12.2, J15.1; no longer J10.2
- new net VBATT_REG: J8.5 (Pin_5), J8.7 (Pin_7), J8.9 (Pin_9)
- no-connect marks 11 -> 17
Other:
- note added: "QWIIC"
- note added: "USB-C Upload/Debugging"
- note added: "X+/Y+/Z+"
- note added: "X-/Y-/Z-"
- note removed: "Power Connectors: USB-C Power Delivery to 2S Li-ion Battery"
- moved on the sheet: J10, J11, J12, J19, J20, J4, J5, J8, JP1
