File: ADCS/ADCS-v01b-samwise/magnetorquer_driver.kicad_sch (KiCad schematic)
At the start: 33 parts, among them U1 MP6551GQB-P, U6 MP6551GQB-P, U8 MP6551GQB-P

Commit message: Changes to ADCS board as of 20250322
Parts:
- C22, C25, C34: value 10u -> 10uF
- C23, C31, C35: value 100n -> 100nF
- C24, C33, C9: value 22u -> 22uF
- C36: renamed from C37; value 3.3u -> 3.3uF
- C40: renamed from C43; value 3.3u -> 3.3uF
- C41: renamed from C44; value 3.3u -> 3.3uF
- C52: renamed from C55; value 3.3u -> 3.3uF
- C53: renamed from C56; value 3.3u -> 3.3uF
- C54: renamed from C57; value 3.3u -> 3.3uF
Changed lines of the file:
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@@
 		(dnp no)
 		(fields_autoplaced yes)
-		(property "Reference" "C44"
+		(property "Reference" "C41"
 			(at 243.84 41.9099 0)
 			(effects
@@
 			)
 		)
-		(property "Value" "3.3u"
+		(property "Value" "3.3uF"
 			(at 243.84 44.4499 0)
 			(effects
@@
 			(project "mainboard"
 				(path "/db20b18b-d25a-428e-8229-70a189e1de75/bf054148-62e0-4cf7-809c-5cbf4e6f48f2"
-					(reference "C44")
+					(reference "C41")
 					(unit 1)
 				)
@@
 			)
 		)
-		(property "Value" "22u"
+		(property "Value" "22uF"
 			(at 29.21 176.5299 0)
 			(effects
@@
 			)
 		)
-		(property "Value" "22u"
+		(property "Value" "22uF"
 			(at 151.13 106.6799 0)
 			(effects
@@
 		(dnp no)
 		(fields_autoplaced yes)
-		(property "Reference" "C55"
+		(property "Reference" "C52"
 			(at 264.16 63.4999 0)
 			(effects
@@
 			)
 		)
-		(property "Value" "3.3u"
+		(property "Value" "3.3uF"
 			(at 264.16 66.0399 0)
 			(effects
@@
 			(project "mainboard"
 				(path "/db20b18b-d25a-428e-8229-70a189e1de75/bf054148-62e0-4cf7-809c-5cbf4e6f48f2"
-					(reference "C55")
+					(reference "C52")
 					(unit 1)
 				)
@@
 			)
 		)
-		(property "Value" "22u"
+		(property "Value" "22uF"
 			(at 27.94 95.2499 0)
 			(effects
@@
 			)
 		)
-		(property "Value" "100n"
+		(property "Value" "100nF"
 			(at 52.07 176.5299 0)
 			(effects
@@
 			)
 		)
-		(property "Value" "100n"
+		(property "Value" "100nF"
 			(at 50.8 95.2499 0)
 			(effects
@@
 		(dnp no)
 		(fields_autoplaced yes)
-		(property "Reference" "C56"
-			(at 119.38 113.0299 0)
+		(property "Reference" "C53"
+			(at 118.491 113.0878 0)
 			(effects
 				(font
@@
 			)
 		)
-		(property "Value" "3.3u"
-			(at 119.38 115.5699 0)
+		(property "Value" "3.3uF"
+			(at 118.491 115.5121 0)
 			(effects
 				(font
@@
 			(project "mainboard"
 				(path "/db20b18b-d25a-428e-8229-70a189e1de75/bf054148-62e0-4cf7-809c-5cbf4e6f48f2"
-					(reference "C56")
+					(reference "C53")
 					(unit 1)
 				)
@@
 		(dnp no)
 		(fields_autoplaced yes)
-		(property "Reference" "C57"
+		(property "Reference" "C54"
 			(at 146.05 133.3499 0)
 			(effects
@@
 			)
 		)
-		(property "Value" "3.3u"
+		(property "Value" "3.3uF"
 			(at 146.05 135.8899 0)
 			(effects
@@
 			(project "mainboard"
 				(path "/db20b18b-d25a-428e-8229-70a189e1de75/bf054148-62e0-4cf7-809c-5cbf4e6f48f2"
-					(reference "C57")
+					(reference "C54")
 					(unit 1)
 				)
@@
 		(dnp no)
 		(fields_autoplaced yes)
-		(property "Reference" "C37"
-			(at 116.84 33.0199 0)
+		(property "Reference" "C36"
+			(at 115.951 33.0778 0)
 			(effects
 				(font
@@
 			)
 		)
-		(property "Value" "3.3u"
-			(at 116.84 35.5599 0)
+		(property "Value" "3.3uF"
+			(at 115.951 35.5021 0)
 			(effects
 				(font
@@
 			(project ""
 				(path "/db20b18b-d25a-428e-8229-70a189e1de75/bf054148-62e0-4cf7-809c-5cbf4e6f48f2"
-					(reference "C37")
+					(reference "C36")
 					(unit 1)
 				)
@@
 			)
 		)
-		(property "Value" "10u"
+		(property "Value" "10uF"
 			(at 40.64 95.2499 0)
 			(effects
@@
 		(dnp no)
 		(fields_autoplaced yes)
-		(property "Reference" "C43"
+		(property "Reference" "C40"
 			(at 139.7 52.0699 0)
 			(effects
@@
 			)
 		)
-		(property "Value" "3.3u"
+		(property "Value" "3.3uF"
 			(at 139.7 54.6099 0)
 			(effects
@@
 			(project "mainboard"
 				(path "/db20b18b-d25a-428e-8229-70a189e1de75/bf054148-62e0-4cf7-809c-5cbf4e6f48f2"
-					(reference "C43")
+					(reference "C40")
 					(unit 1)
 				)
@@
 			)
 		)
-		(property "Value" "10u"
+		(property "Value" "10uF"
 			(at 163.83 106.6799 0)
 			(effects
@@
 			)
 		)
-		(property "Value" "100n"
+		(property "Value" "100nF"
 			(at 173.99 106.6799 0)
 			(effects
@@
 			)
 		)
-		(property "Value" "10u"
+		(property "Value" "10uF"
 			(at 41.91 176.5299 0)
 			(effects
