File: ADCS/ADCS-v01b-samwise/power_enable.kicad_sch (KiCad schematic)
At the start: 5 parts, among them Q1 DMP2040USS-13

Commit message: Changes to ADCS board as of 20250322
Parts:
- C64: renamed from C78; symbol pycubed_mainboard:10NF_10000PF-50V-10%(0603) -> Device:C
- C65: renamed from C79; symbol pycubed_mainboard:10NF_10000PF-50V-10%(0603) -> Device:C
- R18: value 4.7K -> 4.7k
- R19: value ${source_resistor} -> 3.3k
