File: ADCS/ADCS-v01b-samwise/watchdog.kicad_sch (KiCad schematic)
At the start: 28 parts, among them U7 TLV1704

Commit message: Changes to ADCS board as of 20250322
Parts:
- C49: renamed from C52; value 0.1uF -> 100nF
- renumbered C41 to C38, C42 to C39, C51 to C48, C53 to C50, C54 to C51, D6 to D2, D7 to D3, R50 to R49, R53 to R50, R54 to R51, R56 to R52, R62 to R53, R63 to R54, R64 to R55, R68 to R56, R82 to R57, R81 to R58, R76 to R59, R77 to R60, R78 to R61, R79 to R62, R80 to R63, R69 to R64, R70 to R65, R75 to R66
Changed lines of the file:
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@@
 		(dnp no)
 		(fields_autoplaced yes)
-		(property "Reference" "R56"
+		(property "Reference" "R52"
 			(at 105.41 111.76 90)
 			(effects
@@
 			(project "mainboard"
 				(path "/db20b18b-d25a-428e-8229-70a189e1de75/a393ea4a-5f4e-4c0f-917f-6d28e91dd546"
-					(reference "R56")
+					(reference "R52")
 					(unit 1)
 				)
@@
 		(dnp no)
 		(fields_autoplaced yes)
-		(property "Reference" "R50"
+		(property "Reference" "R49"
 			(at 45.72 114.3 90)
 			(effects
@@
 			(project ""
 				(path "/db20b18b-d25a-428e-8229-70a189e1de75/a393ea4a-5f4e-4c0f-917f-6d28e91dd546"
-					(reference "R50")
+					(reference "R49")
 					(unit 1)
 				)
@@
 		(dnp no)
 		(fields_autoplaced yes)
-		(property "Reference" "C51"
+		(property "Reference" "C48"
 			(at 171.45 125.7299 0)
 			(effects
@@
 			(project "mainboard"
 				(path "/db20b18b-d25a-428e-8229-70a189e1de75/a393ea4a-5f4e-4c0f-917f-6d28e91dd546"
-					(reference "C51")
+					(reference "C48")
 					(unit 1)
 				)
@@
 		(dnp no)
 		(fields_autoplaced yes)
-		(property "Reference" "R79"
+		(property "Reference" "R62"
 			(at 101.6 74.9299 0)
 			(effects
@@
 			(project "mainboard"
 				(path "/db20b18b-d25a-428e-8229-70a189e1de75/a393ea4a-5f4e-4c0f-917f-6d28e91dd546"
-					(reference "R79")
+					(reference "R62")
 					(unit 1)
 				)
@@
 		(dnp no)
 		(fields_autoplaced yes)
-		(property "Reference" "C52"
+		(property "Reference" "C49"
 			(at 73.66 49.5299 0)
 			(effects
@@
 			)
 		)
-		(property "Value" "0.1uF"
+		(property "Value" "100nF"
 			(at 73.66 52.0699 0)
 			(effects
@@
 			(project "mainboard"
 				(path "/db20b18b-d25a-428e-8229-70a189e1de75/a393ea4a-5f4e-4c0f-917f-6d28e91dd546"
-					(reference "C52")
+					(reference "C49")
 					(unit 1)
 				)
@@
 		(dnp no)
 		(fields_autoplaced yes)
-		(property "Reference" "R68"
+		(property "Reference" "R56"
 			(at 184.15 134.62 90)
 			(effects
@@
 			(project "mainboard"
 				(path "/db20b18b-d25a-428e-8229-70a189e1de75/a393ea4a-5f4e-4c0f-917f-6d28e91dd546"
-					(reference "R68")
+					(reference "R56")
 					(unit 1)
 				)
@@
 		(dnp no)
 		(fields_autoplaced yes)
-		(property "Reference" "R76"
+		(property "Reference" "R59"
 			(at 101.6 44.4499 0)
 			(effects
@@
 			(project ""
 				(path "/db20b18b-d25a-428e-8229-70a189e1de75/a393ea4a-5f4e-4c0f-917f-6d28e91dd546"
-					(reference "R76")
+					(reference "R59")
 					(unit 1)
 				)
@@
 		(dnp no)
 		(fields_autoplaced yes)
-		(property "Reference" "R69"
+		(property "Reference" "R64"
 			(at 189.23 87.63 90)
 			(effects
@@
 			(project "mainboard"
 				(path "/db20b18b-d25a-428e-8229-70a189e1de75/a393ea4a-5f4e-4c0f-917f-6d28e91dd546"
-					(reference "R69")
+					(reference "R64")
 					(unit 1)
 				)
@@
 		(dnp no)
 		(fields_autoplaced yes)
-		(property "Reference" "D6"
+		(property "Reference" "D2"
 			(at 194.31 134.62 0)
 			(effects
@@
 			(project ""
 				(path "/db20b18b-d25a-428e-8229-70a189e1de75/a393ea4a-5f4e-4c0f-917f-6d28e91dd546"
-					(reference "D6")
+					(reference "D2")
 					(unit 1)
 				)
@@
 		(dnp no)
 		(fields_autoplaced yes)
-		(property "Reference" "R81"
+		(property "Reference" "R58"
 			(at 43.18 35.56 90)
 			(effects
@@
 			(project ""
 				(path "/db20b18b-d25a-428e-8229-70a189e1de75/a393ea4a-5f4e-4c0f-917f-6d28e91dd546"
-					(reference "R81")
+					(reference "R58")
 					(unit 1)
 				)
@@
 		(dnp no)
 		(fields_autoplaced yes)
-		(property "Reference" "C53"
+		(property "Reference" "C50"
 			(at 57.15 49.5299 0)
 			(effects
@@
 			(project ""
 				(path "/db20b18b-d25a-428e-8229-70a189e1de75/a393ea4a-5f4e-4c0f-917f-6d28e91dd546"
-					(reference "C53")
+					(reference "C50")
 					(unit 1)
 				)
@@
 		(dnp no)
 		(fields_autoplaced yes)
-		(property "Reference" "R54"
+		(property "Reference" "R51"
 			(at 66.04 126.9999 0)
 			(effects
@@
 			(project "mainboard"
 				(path "/db20b18b-d25a-428e-8229-70a189e1de75/a393ea4a-5f4e-4c0f-917f-6d28e91dd546"
-					(reference "R54")
+					(reference "R51")
 					(unit 1)
 				)
@@
 		(dnp no)
 		(fields_autoplaced yes)
-		(property "Reference" "C42"
-			(at 160.02 125.7299 0)
+		(property "Reference" "C39"
+			(at 159.131 125.7878 0)
 			(effects
 				(font
@@
 		)
 		(property "Value" "10uF"
-			(at 160.02 128.2699 0)
+			(at 159.131 128.2121 0)
 			(effects
 				(font
@@
 			(project "mainboard"
 				(path "/db20b18b-d25a-428e-8229-70a189e1de75/a393ea4a-5f4e-4c0f-917f-6d28e91dd546"
-					(reference "C42")
+					(reference "C39")
 					(unit 1)
 				)
@@
 		(dnp no)
 		(fields_autoplaced yes)
-		(property "Reference" "R78"
+		(property "Reference" "R61"
 			(at 101.6 64.7699 0)
 			(effects
@@
 			(project "mainboard"
 				(path "/db20b18b-d25a-428e-8229-70a189e1de75/a393ea4a-5f4e-4c0f-917f-6d28e91dd546"
-					(reference "R78")
+					(reference "R61")
 					(unit 1)
 				)
@@
 		(dnp no)
 		(fields_autoplaced yes)
-		(property "Reference" "R70"
+		(property "Reference" "R65"
 			(at 184.15 80.0099 0)
 			(effects
@@
 			(project "mainboard"
 				(path "/db20b18b-d25a-428e-8229-70a189e1de75/a393ea4a-5f4e-4c0f-917f-6d28e91dd546"
-					(reference "R70")
+					(reference "R65")
 					(unit 1)
 				)
@@
 		(dnp no)
 		(fields_autoplaced yes)
-		(property "Reference" "R80"
+		(property "Reference" "R63"
 			(at 101.6 85.0899 0)
 			(effects
@@
 			(project "mainboard"
 				(path "/db20b18b-d25a-428e-8229-70a189e1de75/a393ea4a-5f4e-4c0f-917f-6d28e91dd546"
-					(reference "R80")
+					(reference "R63")
 					(unit 1)
 				)
@@
 		(dnp no)
 		(fields_autoplaced yes)
-		(property "Reference" "R77"
+		(property "Reference" "R60"
 			(at 101.6 54.6099 0)
 			(effects
@@
 			(project "mainboard"
 				(path "/db20b18b-d25a-428e-8229-70a189e1de75/a393ea4a-5f4e-4c0f-917f-6d28e91dd546"
-					(reference "R77")
+					(reference "R60")
 					(unit 1)
 				)
@@
 		(dnp no)
 		(fields_autoplaced yes)
-		(property "Reference" "R82"
+		(property "Reference" "R57"
 			(at 246.38 114.3 90)
 			(effects
@@
 			(project "mainboard"
 				(path "/db20b18b-d25a-428e-8229-70a189e1de75/a393ea4a-5f4e-4c0f-917f-6d28e91dd546"
-					(reference "R82")
+					(reference "R57")
 					(unit 1)
 				)
@@
 		(dnp no)
 		(fields_autoplaced yes)
-		(property "Reference" "C41"
-			(at 118.11 124.4599 0)
+		(property "Reference" "C38"
+			(at 117.221 124.5178 0)
 			(effects
 				(font
@@
 		)
 		(property "Value" "10uF"
-			(at 118.11 126.9999 0)
+			(at 117.221 126.9421 0)
 			(effects
 				(font
@@
 			(project "mainboard"
 				(path "/db20b18b-d25a-428e-8229-70a189e1de75/a393ea4a-5f4e-4c0f-917f-6d28e91dd546"
-					(reference "C41")
+					(reference "C38")
 					(unit 1)
 				)
@@
 		(dnp no)
 		(fields_autoplaced yes)
-		(property "Reference" "R53"
+		(property "Reference" "R50"
 			(at 69.85 114.3 90)
 			(effects
@@
 			(project "mainboard"
 				(path "/db20b18b-d25a-428e-8229-70a189e1de75/a393ea4a-5f4e-4c0f-917f-6d28e91dd546"
-					(reference "R53")
+					(reference "R50")
 					(unit 1)
 				)
@@
 		(dnp no)
 		(fields_autoplaced yes)
-		(property "Reference" "R64"
+		(property "Reference" "R55"
 			(at 190.5 124.46 90)
 			(effects
@@
 			(project "mainboard"
 				(path "/db20b18b-d25a-428e-8229-70a189e1de75/a393ea4a-5f4e-4c0f-917f-6d28e91dd546"
-					(reference "R64")
+					(reference "R55")
 					(unit 1)
 				)
@@
 		(dnp no)
 		(fields_autoplaced yes)
-		(property "Reference" "D7"
+		(property "Reference" "D3"
 			(at 30.7975 35.56 0)
 			(effects
@@
 			(project ""
 				(path "/db20b18b-d25a-428e-8229-70a189e1de75/a393ea4a-5f4e-4c0f-917f-6d28e91dd546"
-					(reference "D7")
+					(reference "D3")
 					(unit 1)
 				)
@@
 		(dnp no)
 		(fields_autoplaced yes)
-		(property "Reference" "R63"
+		(property "Reference" "R54"
 			(at 149.86 114.3 90)
 			(effects
@@
 			(project ""
 				(path "/db20b18b-d25a-428e-8229-70a189e1de75/a393ea4a-5f4e-4c0f-917f-6d28e91dd546"
-					(reference "R63")
+					(reference "R54")
 					(unit 1)
 				)
@@
 		(dnp no)
 		(fields_autoplaced yes)
-		(property "Reference" "R75"
+		(property "Reference" "R66"
 			(at 203.2 80.0099 0)
 			(effects
@@
 			(project "mainboard"
 				(path "/db20b18b-d25a-428e-8229-70a189e1de75/a393ea4a-5f4e-4c0f-917f-6d28e91dd546"
-					(reference "R75")
+					(reference "R66")
 					(unit 1)
 				)
@@
 		(dnp no)
 		(fields_autoplaced yes)
-		(property "Reference" "R62"
+		(property "Reference" "R53"
 			(at 116.84 107.9499 0)
 			(effects
@@
 			(project "mainboard"
 				(path "/db20b18b-d25a-428e-8229-70a189e1de75/a393ea4a-5f4e-4c0f-917f-6d28e91dd546"
-					(reference "R62")
+					(reference "R53")
 					(unit 1)
 				)
@@
 		(dnp no)
 		(fields_autoplaced yes)
-		(property "Reference" "C54"
+		(property "Reference" "C51"
 			(at 227.33 82.5499 0)
 			(effects
@@
 			(project "mainboard"
 				(path "/db20b18b-d25a-428e-8229-70a189e1de75/a393ea4a-5f4e-4c0f-917f-6d28e91dd546"
-					(reference "C54")
+					(reference "C51")
 					(unit 1)
 				)
