File: ADCS/ADCS-v01b-samwise/GPS.kicad_sch (KiCad schematic)
At the start: 5 parts, among them J6 Amphenol_901-144, J7 Amphenol_901-144, U12 Orion B16, U13 EP2W+

Commit message: Updated ADCS board to KiCad 9, cleaned up 3D models
Parts:
- J6, J7: footprint Connector_Coaxial:SMA_Amphenol_901-144_Vertical -> ssi_connector:SMA_Amphenol_901-144_horizontal
Changed lines of the file:
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@@
 			)
 		)
-		(property "Footprint" "Connector_Coaxial:SMA_Amphenol_901-144_Vertical"
+		(property "Footprint" "ssi_connector:SMA_Amphenol_901-144_horizontal"
 			(at 241.3 71.12 0)
 			(effects
@@
 			)
 		)
-		(property "Footprint" "Connector_Coaxial:SMA_Amphenol_901-144_Vertical"
+		(property "Footprint" "ssi_connector:SMA_Amphenol_901-144_horizontal"
 			(at 241.3 60.96 0)
 			(effects
