File: PiCubed/MPPT_addon_board/I2C_Bus_Protection.kicad_sch (KiCad schematic)
At the start: 18 parts, among them Q1 BSS138DWQ-7, Q2 MBT2222ADW1T1, Q3 BSS138DWQ-7, Q4 MBT2222ADW1T1

Commit message: Updated MPPT add-on board to Kicad 9
Parts:
- Q2, Q4: Flight MBT2222ADW1T1G -> MBT2222ADW1T1; Manufacturer_Part_Number MBT2222ADW1T1G -> MBT2222ADW1T1; Proto MBT2222ADW1T1G -> MBT2222ADW1T1
