File: ADCS/ADCS-v1-samwise/imu_and_magnetometer.kicad_sch (KiCad schematic)
At the start: 3 parts, among them U10 RM3100CB, U11 BMI270

Commit message: ver 1.5
Other:
- note added: "Magnetometer"
- note removed: "Magnetometers"
Changed lines of the file:
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@@
 		(title "ADCS Main Board")
 		(date "2025-05-21")
-		(rev "1.4")
+		(rev "1.5")
 		(company "Stanford Student Space Initiative")
 		(comment 1 "Sage Wu")
@@
 		)
 	)
-	(text "Magnetometers"
+	(text "Magnetometer"
 		(exclude_from_sim no)
 		(at 113.03 65.024 0)
@@
 					(size 1.27 1.27)
 				)
+				(hide yes)
 			)
 		)
@@
 					(size 1.27 1.27)
 				)
-			)
-		)
+				(hide yes)
+			)
+		)

Commit message: ADCS v1.7
Parts:
- removed U10: RM3100CB, ssi_IC:RM3100CB, symbol ssi_IC:RM3100-CB_AliExpress
- added U10: RM3100CB, ssi_IC:RM3100CB, symbol ssi_IC:RM3100-CB
Connections:
- net 3V3_MAGNMETER: now also U10.5 (VCC)
- net GND: now also U10.4 (GND)
- net MAGMETER_DRDY: now also U10.7 (DRDY)
- net MISO_MAGMETER: now also U10.2 (MISO)
- net MOSI_MAGMETER: now also U10.3 (MOSI)
- net SCLK_MAGMETER: now also U10.1 (SLCK)
- net SCS_MAGMETER: now also U10.6 (SCS)
Changed lines of the file:
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@@
 		(title "ADCS Main Board")
 		(date "2025-05-22")
-		(rev "1.6")
+		(rev "1.7")
 		(company "Stanford Student Space Initiative")
 		(comment 1 "Sage Wu")
@@
 	)
 	(symbol
+		(lib_id "ssi_IC:RM3100-CB")
+		(at 113.03 82.55 0)
+		(unit 1)
+		(exclude_from_sim no)
+		(in_bom yes)
+		(on_board yes)
+		(dnp no)
+		(fields_autoplaced yes)
+		(property "Reference" "U10"
+			(at 113.03 69.85 0)
+			(effects
+				(font
+					(size 1.27 1.27)
+				)
+			)
+		)
+		(property "Value" "RM3100CB"
+			(at 113.03 72.39 0)
+			(effects
+				(font
+					(size 1.27 1.27)
+				)
+			)
+		)
+		(property "Footprint" "ssi_IC:RM3100CB"
+			(at 113.03 91.694 0)
+			(effects
+				(font
+					(size 1.27 1.27)
+				)
+				(hide yes)
+			)
+		)
+		(property "Datasheet" "https://www.pnisensor.com/rm3100-cb/#download-rm3100-cb-manual"
+			(at 113.03 82.55 0)
+			(effects
+				(font
+					(size 1.27 1.27)
+				)
+				(hide yes)
+			)
+		)
+		(property "Description" ""
+			(at 113.03 82.55 0)
+			(effects
+				(font
+					(size 1.27 1.27)
+				)
+				(hide yes)
+			)
+		)
+		(property "Height" ""
+			(at 113.03 82.55 0)
+			(effects
+				(font
+					(size 1.27 1.27)
+				)
+				(hide yes)
+			)
+		)
+		(pin "8"
+		)
+		(pin "3"
+		)
+		(pin "4"
+		)
+		(pin "5"
+		)
+		(pin "6"
+		)
+		(pin "7"
+		)
+		(pin "1"
+		)
+		(pin "2"
+		)
+		(instances
+			(project ""
+				(path "/db20b18b-d25a-428e-8229-70a189e1de75/a3d832b6-a1cc-4410-a8d7-1698d429804f"
+					(reference "U10")
+					(unit 1)
+				)
+			)
+		)
+	)
+	(symbol
 		(lib_id "power:+3V3")
 		(at 48.26 127 0)
@@
 					(unit 1)
 				)
-			)
-		)
-	)
-	(symbol
-		(lib_id "ssi_IC:RM3100-CB_AliExpress")
-		(at 113.03 82.55 0)
-		(unit 1)
-		(exclude_from_sim no)
-		(in_bom yes)
-		(on_board yes)
-		(dnp no)
-		(fields_autoplaced yes)
-		(property "Reference" "U10"
-			(at 113.03 70.9125 0)
-			(effects
-				(font
-					(size 1.27 1.27)
-				)
-			)
-		)
-		(property "Value" "RM3100CB"
-			(at 113.03 73.3368 0)
-			(effects
-				(font
-					(size 1.27 1.27)
-				)
-			)
-		)
-		(property "Footprint" "ssi_IC:RM3100CB"
-			(at 113.03 91.694 0)
-			(effects
-				(font
-					(size 1.27 1.27)
-				)
-				(hide yes)
-			)
-		)
-		(property "Datasheet" "https://www.pnisensor.com/rm3100-cb/#download-rm3100-cb-manual"
-			(at 113.03 82.55 0)
-			(effects
-				(font
-					(size 1.27 1.27)
-				)
-				(hide yes)
-			)
-		)
-		(property "Description" ""
-			(at 113.03 82.55 0)
-			(effects
-				(font
-					(size 1.27 1.27)
-				)
-				(hide yes)
-			)
-		)
-		(property "Height" ""
-			(at 113.03 82.55 0)
-			(effects
-				(font
-					(size 1.27 1.27)
-				)
-				(hide yes)
-			)
-		)
-		(pin "6"
-		)
-		(pin "3"
-		)
-		(pin "8"
-		)
-		(pin "2"
-		)
-		(pin "7"
-		)
-		(pin "1"
-		)
-		(pin "5"
-		)
-		(pin "4"
-		)
-		(instances
-			(project "mainboard"
-				(path "/db20b18b-d25a-428e-8229-70a189e1de75/a3d832b6-a1cc-4410-a8d7-1698d429804f"
-					(reference "U10")
-					(unit 1)
-				)
